Commit message: building ros_wrapper

File: a1_robot/urdf/a1.urdf (robot description, URDF)
Before this commit: robot a1_description, 23 links, 22 joints
Links:
- removed link FL_calf
- removed link FL_foot
- removed link FL_thigh
- removed link FL_thigh_shoulder
- removed link FR_calf
- removed link FR_foot
- removed link FR_thigh
- removed link FR_thigh_shoulder
- removed link RL_calf
- removed link RL_foot
- removed link RL_thigh
- removed link RL_thigh_shoulder
- removed link RR_calf
- removed link RR_foot
- removed link RR_thigh
- removed link RR_thigh_shoulder
- removed link base
- added link FL_lower, mass 0.166; collision box size=0.2 0.016 0.016; visual mesh filename=meshes/calf.obj scale=1 1 1
- added link FL_toe, mass 0.06; collision sphere radius=0.02; visual sphere radius=0.01
- added link FL_upper, mass 1.013; collision box size=0.2 0.0245 0.034; visual mesh filename=meshes/thigh.obj scale=1 1 1
- added link FL_upper_shoulder, mass 0.001; collision cylinder length=0.032 radius=0.041; visual cylinder length=0.032 radius=0.040
- added link FR_lower, mass 0.166; collision box size=0.2 0.016 0.016; visual mesh filename=meshes/calf.obj scale=1 1 1
- added link FR_toe, mass 0.06; collision sphere radius=0.02; visual sphere radius=0.01
- added link FR_upper, mass 1.013; collision box size=0.2 0.0245 0.034; visual mesh filename=meshes/thigh_mirror.obj scale=1 1 1
- added link FR_upper_shoulder, mass 0.001; collision cylinder length=0.032 radius=0.041; visual cylinder length=0.032 radius=0.040
- added link RL_lower, mass 0.166; collision box size=0.2 0.016 0.016; visual mesh filename=meshes/calf.obj scale=1 1 1
- added link RL_toe, mass 0.06; collision sphere radius=0.02; visual sphere radius=0.01
- added link RL_upper, mass 1.013; collision box size=0.2 0.0245 0.034; visual mesh filename=meshes/thigh.obj scale=1 1 1
- added link RL_upper_shoulder, mass 0.001; collision cylinder length=0.032 radius=0.041; visual cylinder length=0.032 radius=0.040
- added link RR_lower, mass 0.166; collision box size=0.2 0.016 0.016; visual mesh filename=meshes/calf.obj scale=1 1 1
- added link RR_toe, mass 0.06; collision sphere radius=0.02; visual sphere radius=0.01
- added link RR_upper, mass 1.013; collision box size=0.2 0.0245 0.034; visual mesh filename=meshes/thigh_mirror.obj scale=1 1 1
- added link RR_upper_shoulder, mass 0.001; collision cylinder length=0.032 radius=0.041; visual cylinder length=0.032 radius=0.040
- link FL_hip: geometry collision cylinder length=0.04 radius=0.046; visual mesh filename=meshes/hip.obj scale=1 1 1
- link FR_hip: geometry collision cylinder length=0.04 radius=0.046; visual mesh filename=meshes/hip.obj scale=1 1 1
- link RL_hip: geometry collision cylinder length=0.04 radius=0.046; visual mesh filename=meshes/hip.obj scale=1 1 1
- link RR_hip: geometry collision cylinder length=0.04 radius=0.046; visual mesh filename=meshes/hip.obj scale=1 1 1
- link trunk: mass 6.0 -> 4.713; geometry collision box size=0.267 0.194 0.114; visual mesh filename=meshes/trunk.obj scale=1 1 1
Joints:
- removed joint floating_base
- joint FL_calf_joint: child FL_calf -> FL_lower; limit lower=-2.69653369433 upper=-0.916297857297 effort=33.5 velocity=21 -> lower=-2.69653369433 upper=-0.916297857297 effort=55 velocity=28.6; parent FL_thigh -> FL_upper
- joint FL_foot_fixed: child FL_foot -> FL_toe; parent FL_calf -> FL_lower
- joint FL_hip_fixed: child FL_thigh_shoulder -> FL_upper_shoulder
- joint FL_hip_joint: limit lower=-0.802851455917 upper=0.802851455917 effort=33.5 velocity=21 -> lower=-0.802851455917 upper=0.802851455917 effort=20 velocity=52.4; origin xyz=0.1805 0.047 0 rpy=0 0 0 -> xyz=0.183 0.047 0 rpy=0 0 0
- joint FL_thigh_joint: child FL_thigh -> FL_upper; limit lower=-1.0471975512 upper=4.18879020479 effort=33.5 velocity=21 -> lower=-1.0471975512 upper=4.18879020479 effort=55 velocity=28.6; origin xyz=0 0.0838 0 rpy=0 0 0 -> xyz=0 0.08505 0 rpy=0 0 0
- joint FR_calf_joint: child FR_calf -> FR_lower; limit lower=-2.69653369433 upper=-0.916297857297 effort=33.5 velocity=21 -> lower=-2.69653369433 upper=-0.916297857297 effort=55 velocity=28.6; parent FR_thigh -> FR_upper
- joint FR_foot_fixed: child FR_foot -> FR_toe; parent FR_calf -> FR_lower
- joint FR_hip_fixed: child FR_thigh_shoulder -> FR_upper_shoulder
- joint FR_hip_joint: limit lower=-0.802851455917 upper=0.802851455917 effort=33.5 velocity=21 -> lower=-0.802851455917 upper=0.802851455917 effort=20 velocity=52.4; origin xyz=0.1805 -0.047 0 rpy=0 0 0 -> xyz=0.183 -0.047 0 rpy=0 0 0
- joint FR_thigh_joint: child FR_thigh -> FR_upper; limit lower=-1.0471975512 upper=4.18879020479 effort=33.5 velocity=21 -> lower=-1.0471975512 upper=4.18879020479 effort=55 velocity=28.6; origin xyz=0 -0.0838 0 rpy=0 0 0 -> xyz=0 -0.08505 0 rpy=0 0 0
- joint RL_calf_joint: child RL_calf -> RL_lower; limit lower=-2.69653369433 upper=-0.916297857297 effort=33.5 velocity=21 -> lower=-2.69653369433 upper=-0.916297857297 effort=55 velocity=28.6; parent RL_thigh -> RL_upper
- joint RL_foot_fixed: child RL_foot -> RL_toe; parent RL_calf -> RL_lower
- joint RL_hip_fixed: child RL_thigh_shoulder -> RL_upper_shoulder
- joint RL_hip_joint: limit lower=-0.802851455917 upper=0.802851455917 effort=33.5 velocity=21 -> lower=-0.802851455917 upper=0.802851455917 effort=20 velocity=52.4; origin xyz=-0.1805 0.047 0 rpy=0 0 0 -> xyz=-0.183 0.047 0 rpy=0 0 0
- joint RL_thigh_joint: child RL_thigh -> RL_upper; limit lower=-1.0471975512 upper=4.18879020479 effort=33.5 velocity=21 -> lower=-1.0471975512 upper=4.18879020479 effort=55 velocity=28.6; origin xyz=0 0.0838 0 rpy=0 0 0 -> xyz=0 0.08505 0 rpy=0 0 0
- joint RR_calf_joint: child RR_calf -> RR_lower; limit lower=-2.69653369433 upper=-0.916297857297 effort=33.5 velocity=21 -> lower=-2.69653369433 upper=-0.916297857297 effort=55 velocity=28.6; parent RR_thigh -> RR_upper
- joint RR_foot_fixed: child RR_foot -> RR_toe; parent RR_calf -> RR_lower
- joint RR_hip_fixed: child RR_thigh_shoulder -> RR_upper_shoulder
- joint RR_hip_joint: limit lower=-0.802851455917 upper=0.802851455917 effort=33.5 velocity=21 -> lower=-0.802851455917 upper=0.802851455917 effort=20 velocity=52.4; origin xyz=-0.1805 -0.047 0 rpy=0 0 0 -> xyz=-0.183 -0.047 0 rpy=0 0 0
- joint RR_thigh_joint: child RR_thigh -> RR_upper; limit lower=-1.0471975512 upper=4.18879020479 effort=33.5 velocity=21 -> lower=-1.0471975512 upper=4.18879020479 effort=55 velocity=28.6; origin xyz=0 -0.0838 0 rpy=0 0 0 -> xyz=0 -0.08505 0 rpy=0 0 0
